File: pcb/downlow/downlow.sch (KiCad schematic (older format))
At the start: 54 parts, among them J1 Conn_01x24_Male, J2 Conn_01x24_Male, J3 Conn_01x04_Male, J4 Conn_01x04_Male, J5 Conn_01x04_Male, J6 Conn_01x04_Male, U2 Teensy4.1

Commit message: Minor updates to PDB.
Parts:
- R1, R10, R11, R12, R2, R3, R4, R5, R6, R7, R8, R9: value R -> 2k
- R13, R14, R15, R16, R25, R26, R27, R28: value R -> 2.2k
- R17, R18, R19, R20, R21, R22, R23, R24: value R -> 3.3k
Changed lines of the file:
@@
 U 1 1 625F0E19
 P 3850 1350
-F 0 "R1" V 3643 1350 50  0000 C CNN
-F 1 "R" V 3734 1350 50  0000 C CNN
+F 0 "R1" V 3850 1500 50  0000 C CNN
+F 1 "2k" V 3850 1350 50  0000 C CNN
 F 2 "Resistor_THT:R_Axial_DIN0207_L6.3mm_D2.5mm_P7.62mm_Horizontal" V 3780 1350 50  0001 C CNN
 F 3 "~" H 3850 1350 50  0001 C CNN
@@
 U 1 1 62603EC6
 P 3850 1450
-F 0 "R2" V 3643 1450 50  0000 C CNN
-F 1 "R" V 3734 1450 50  0000 C CNN
+F 0 "R2" V 3850 1600 50  0000 C CNN
+F 1 "2k" V 3850 1450 50  0000 C CNN
 F 2 "Resistor_THT:R_Axial_DIN0207_L6.3mm_D2.5mm_P7.62mm_Horizontal" V 3780 1450 50  0001 C CNN
 F 3 "~" H 3850 1450 50  0001 C CNN
@@
 U 1 1 6260497E
 P 3850 1550
-F 0 "R3" V 3643 1550 50  0000 C CNN
-F 1 "R" V 3734 1550 50  0000 C CNN
+F 0 "R3" V 3850 1700 50  0000 C CNN
+F 1 "2k" V 3850 1550 50  0000 C CNN
 F 2 "Resistor_THT:R_Axial_DIN0207_L6.3mm_D2.5mm_P7.62mm_Horizontal" V 3780 1550 50  0001 C CNN
 F 3 "~" H 3850 1550 50  0001 C CNN
@@
 U 1 1 62605479
 P 3850 1650
-F 0 "R4" V 3643 1650 50  0000 C CNN
-F 1 "R" V 3734 1650 50  0000 C CNN
+F 0 "R4" V 3850 1800 50  0000 C CNN
+F 1 "2k" V 3850 1650 50  0000 C CNN
 F 2 "Resistor_THT:R_Axial_DIN0207_L6.3mm_D2.5mm_P7.62mm_Horizontal" V 3780 1650 50  0001 C CNN
 F 3 "~" H 3850 1650 50  0001 C CNN
@@
 U 1 1 62609A63
 P 3850 1750
-F 0 "R5" V 3643 1750 50  0000 C CNN
-F 1 "R" V 3734 1750 50  0000 C CNN
+F 0 "R5" V 3850 1900 50  0000 C CNN
+F 1 "2k" V 3850 1750 50  0000 C CNN
 F 2 "Resistor_THT:R_Axial_DIN0207_L6.3mm_D2.5mm_P7.62mm_Horizontal" V 3780 1750 50  0001 C CNN
 F 3 "~" H 3850 1750 50  0001 C CNN
@@
 U 1 1 6260B896
 P 3850 1950
-F 0 "R6" V 3643 1950 50  0000 C CNN
-F 1 "R" V 3734 1950 50  0000 C CNN
+F 0 "R6" V 3850 2100 50  0000 C CNN
+F 1 "2k" V 3850 1950 50  0000 C CNN
 F 2 "Resistor_THT:R_Axial_DIN0207_L6.3mm_D2.5mm_P7.62mm_Horizontal" V 3780 1950 50  0001 C CNN
 F 3 "~" H 3850 1950 50  0001 C CNN
@@
 U 1 1 6260C2F4
 P 3850 3350
-F 0 "R12" V 3643 3350 50  0000 C CNN
-F 1 "R" V 3734 3350 50  0000 C CNN
+F 0 "R12" V 3850 3550 50  0000 C CNN
+F 1 "2k" V 3850 3350 50  0000 C CNN
 F 2 "Resistor_THT:R_Axial_DIN0207_L6.3mm_D2.5mm_P7.62mm_Horizontal" V 3780 3350 50  0001 C CNN
 F 3 "~" H 3850 3350 50  0001 C CNN
@@
 U 1 1 6260F5CA
 P 3850 3250
-F 0 "R11" V 3643 3250 50  0000 C CNN
-F 1 "R" V 3734 3250 50  0000 C CNN
+F 0 "R11" V 3850 3450 50  0000 C CNN
+F 1 "2k" V 3850 3250 50  0000 C CNN
 F 2 "Resistor_THT:R_Axial_DIN0207_L6.3mm_D2.5mm_P7.62mm_Horizontal" V 3780 3250 50  0001 C CNN
 F 3 "~" H 3850 3250 50  0001 C CNN
@@
 U 1 1 6262C4F4
 P 3850 2450
-F 0 "R10" V 3643 2450 50  0000 C CNN
-F 1 "R" V 3734 2450 50  0000 C CNN
+F 0 "R10" V 3850 2650 50  0000 C CNN
+F 1 "2k" V 3850 2450 50  0000 C CNN
 F 2 "Resistor_THT:R_Axial_DIN0207_L6.3mm_D2.5mm_P7.62mm_Horizontal" V 3780 2450 50  0001 C CNN
 F 3 "~" H 3850 2450 50  0001 C CNN
@@
 U 1 1 6262D074
 P 3850 2350
-F 0 "R9" V 3643 2350 50  0000 C CNN
-F 1 "R" V 3734 2350 50  0000 C CNN
+F 0 "R9" V 3850 2500 50  0000 C CNN
+F 1 "2k" V 3850 2350 50  0000 C CNN
 F 2 "Resistor_THT:R_Axial_DIN0207_L6.3mm_D2.5mm_P7.62mm_Horizontal" V 3780 2350 50  0001 C CNN
 F 3 "~" H 3850 2350 50  0001 C CNN
@@
 U 1 1 6262DCAB
 P 3850 2250
-F 0 "R8" V 3643 2250 50  0000 C CNN
-F 1 "R" V 3734 2250 50  0000 C CNN
+F 0 "R8" V 3850 2400 50  0000 C CNN
+F 1 "2k" V 3850 2250 50  0000 C CNN
 F 2 "Resistor_THT:R_Axial_DIN0207_L6.3mm_D2.5mm_P7.62mm_Horizontal" V 3780 2250 50  0001 C CNN
 F 3 "~" H 3850 2250 50  0001 C CNN
@@
 U 1 1 6262E959
 P 3850 2150
-F 0 "R7" V 3643 2150 50  0000 C CNN
-F 1 "R" V 3734 2150 50  0000 C CNN
+F 0 "R7" V 3850 2300 50  0000 C CNN
+F 1 "2k" V 3850 2150 50  0000 C CNN
 F 2 "Resistor_THT:R_Axial_DIN0207_L6.3mm_D2.5mm_P7.62mm_Horizontal" V 3780 2150 50  0001 C CNN
 F 3 "~" H 3850 2150 50  0001 C CNN
@@
 P 2650 6300
 F 0 "R16" V 2443 6300 50  0000 C CNN
-F 1 "R" V 2534 6300 50  0000 C CNN
+F 1 "2.2k" V 2534 6300 50  0000 C CNN
 F 2 "Resistor_THT:R_Axial_DIN0207_L6.3mm_D2.5mm_P7.62mm_Horizontal" V 2580 6300 50  0001 C CNN
 F 3 "~" H 2650 6300 50  0001 C CNN
@@
 P 2650 5750
 F 0 "R15" V 2443 5750 50  0000 C CNN
-F 1 "R" V 2534 5750 50  0000 C CNN
+F 1 "2.2k" V 2534 5750 50  0000 C CNN
 F 2 "Resistor_THT:R_Axial_DIN0207_L6.3mm_D2.5mm_P7.62mm_Horizontal" V 2580 5750 50  0001 C CNN
 F 3 "~" H 2650 5750 50  0001 C CNN
@@
 P 2650 5200
 F 0 "R14" V 2443 5200 50  0000 C CNN
-F 1 "R" V 2534 5200 50  0000 C CNN
+F 1 "2.2k" V 2534 5200 50  0000 C CNN
 F 2 "Resistor_THT:R_Axial_DIN0207_L6.3mm_D2.5mm_P7.62mm_Horizontal" V 2580 5200 50  0001 C CNN
 F 3 "~" H 2650 5200 50  0001 C CNN
@@
 P 2650 4700
 F 0 "R13" V 2443 4700 50  0000 C CNN
-F 1 "R" V 2534 4700 50  0000 C CNN
+F 1 "2.2k" V 2534 4700 50  0000 C CNN
 F 2 "Resistor_THT:R_Axial_DIN0207_L6.3mm_D2.5mm_P7.62mm_Horizontal" V 2580 4700 50  0001 C CNN
 F 3 "~" H 2650 4700 50  0001 C CNN
@@
 P 3000 4700
 F 0 "R17" V 2793 4700 50  0000 C CNN
-F 1 "R" V 2884 4700 50  0000 C CNN
+F 1 "3.3k" V 2884 4700 50  0000 C CNN
 F 2 "Resistor_THT:R_Axial_DIN0207_L6.3mm_D2.5mm_P7.62mm_Horizontal" V 2930 4700 50  0001 C CNN
 F 3 "~" H 3000 4700 50  0001 C CNN
@@
 P 3000 5200
 F 0 "R18" V 2793 5200 50  0000 C CNN
-F 1 "R" V 2884 5200 50  0000 C CNN
+F 1 "3.3k" V 2884 5200 50  0000 C CNN
 F 2 "Resistor_THT:R_Axial_DIN0207_L6.3mm_D2.5mm_P7.62mm_Horizontal" V 2930 5200 50  0001 C CNN
 F 3 "~" H 3000 5200 50  0001 C CNN
@@
 P 3000 5750
 F 0 "R19" V 2793 5750 50  0000 C CNN
-F 1 "R" V 2884 5750 50  0000 C CNN
+F 1 "3.3k" V 2884 5750 50  0000 C CNN
 F 2 "Resistor_THT:R_Axial_DIN0207_L6.3mm_D2.5mm_P7.62mm_Horizontal" V 2930 5750 50  0001 C CNN
 F 3 "~" H 3000 5750 50  0001 C CNN
@@
 P 3000 6300
 F 0 "R20" V 2793 6300 50  0000 C CNN
-F 1 "R" V 2884 6300 50  0000 C CNN
+F 1 "3.3k" V 2884 6300 50  0000 C CNN
 F 2 "Resistor_THT:R_Axial_DIN0207_L6.3mm_D2.5mm_P7.62mm_Horizontal" V 2930 6300 50  0001 C CNN
 F 3 "~" H 3000 6300 50  0001 C CNN
@@
 P 7700 5350
 F 0 "R28" V 7493 5350 50  0000 C CNN
-F 1 "R" V 7584 5350 50  0000 C CNN
+F 1 "2.2k" V 7584 5350 50  0000 C CNN
 F 2 "Resistor_THT:R_Axial_DIN0207_L6.3mm_D2.5mm_P7.62mm_Horizontal" V 7630 5350 50  0001 C CNN
 F 3 "~" H 7700 5350 50  0001 C CNN
@@
 P 7300 5350
 F 0 "R24" V 7093 5350 50  0000 C CNN
-F 1 "R" V 7184 5350 50  0000 C CNN
+F 1 "3.3k" V 7184 5350 50  0000 C CNN
 F 2 "Resistor_THT:R_Axial_DIN0207_L6.3mm_D2.5mm_P7.62mm_Horizontal" V 7230 5350 50  0001 C CNN
 F 3 "~" H 7300 5350 50  0001 C CNN
@@
 P 7300 4850
 F 0 "R23" V 7093 4850 50  0000 C CNN
-F 1 "R" V 7184 4850 50  0000 C CNN
+F 1 "3.3k" V 7184 4850 50  0000 C CNN
 F 2 "Resistor_THT:R_Axial_DIN0207_L6.3mm_D2.5mm_P7.62mm_Horizontal" V 7230 4850 50  0001 C CNN
 F 3 "~" H 7300 4850 50  0001 C CNN
@@
 P 7700 4850
 F 0 "R27" V 7493 4850 50  0000 C CNN
-F 1 "R" V 7584 4850 50  0000 C CNN
+F 1 "2.2k" V 7584 4850 50  0000 C CNN
 F 2 "Resistor_THT:R_Axial_DIN0207_L6.3mm_D2.5mm_P7.62mm_Horizontal" V 7630 4850 50  0001 C CNN
 F 3 "~" H 7700 4850 50  0001 C CNN
@@
 P 7700 4400
 F 0 "R26" V 7493 4400 50  0000 C CNN
-F 1 "R" V 7584 4400 50  0000 C CNN
+F 1 "2.2k" V 7584 4400 50  0000 C CNN
 F 2 "Resistor_THT:R_Axial_DIN0207_L6.3mm_D2.5mm_P7.62mm_Horizontal" V 7630 4400 50  0001 C CNN
 F 3 "~" H 7700 4400 50  0001 C CNN
@@
 P 7300 4400
 F 0 "R22" V 7093 4400 50  0000 C CNN
-F 1 "R" V 7184 4400 50  0000 C CNN
+F 1 "3.3k" V 7184 4400 50  0000 C CNN
 F 2 "Resistor_THT:R_Axial_DIN0207_L6.3mm_D2.5mm_P7.62mm_Horizontal" V 7230 4400 50  0001 C CNN
 F 3 "~" H 7300 4400 50  0001 C CNN
@@
 P 7300 3950
 F 0 "R21" V 7093 3950 50  0000 C CNN
-F 1 "R" V 7184 3950 50  0000 C CNN
+F 1 "3.3k" V 7184 3950 50  0000 C CNN
 F 2 "Resistor_THT:R_Axial_DIN0207_L6.3mm_D2.5mm_P7.62mm_Horizontal" V 7230 3950 50  0001 C CNN
 F 3 "~" H 7300 3950 50  0001 C CNN
@@
 P 7700 3950
 F 0 "R25" V 7493 3950 50  0000 C CNN
-F 1 "R" V 7584 3950 50  0000 C CNN
+F 1 "2.2k" V 7584 3950 50  0000 C CNN
 F 2 "Resistor_THT:R_Axial_DIN0207_L6.3mm_D2.5mm_P7.62mm_Horizontal" V 7630 3950 50  0001 C CNN
 F 3 "~" H 7700 3950 50  0001 C CNN
