File: pcb/downlow/downlow.kicad_pcb (KiCad board)
At the start: 4 copper layers, 64.8 x 76.2 mm, 59 parts, among them J1 Conn_01x24_Male, J2 Conn_01x24_Male, J3 Conn_01x04_Male, J4 Conn_01x04_Male, J5 Conn_01x04_Male, J6 Conn_01x04_Male, M3 MountingHole_3.2mm_M3_ISO1458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, U2 Teensy4.1

Commit message: Update PCB files for new KiCAD version.
Other:
- net class Default removed
